File: pizero-papoe/pizero-papoe.kicad_pcb (KiCad board)
At the start: 4 copper layers, 80 x 30 mm, 97 parts, among them IC1 RTL8153B-VB-CG, J1 PogoPin_01x01, J2 PogoPin_01x01, J3 PogoPin_01x01, J4 PogoPin_01x01, J5 PogoPin_01x01, J6 RJ45_LED_AK_Shielded, P1 USB_C_Plug_USB3.0_9P, Q2 DMMT3906_Dual_PNP, Q3 Q_PMOS_GSD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

Commit message: pizero-papoe pcb sch bom tweaks for r1
Parts:
- added D11: LED Green, LED_SMD:LED_0603_1608Metric, F.Cu at (97.3, 82.7)
- added F2: JFC1206-1250FS, Fuse:Fuse_1206_3216Metric, F.Cu at (121.8, 81.7)
- added R9: 10k, Resistor_SMD:R_0603_1608Metric, F.Cu at (102.6, 82.7)
- C1, C10, C25, C26, C27, C28, C30, C31, C33, C35, C36, C41, C42, C7, C8, C9: value 0.1uf -> 0.1uF
- C2, C3: value 30pf -> 30pF
- C23, C24: value nostuff-330-1200uF -> 330-1200uF-dnp
- D3: value SMAJ58A -> SMAJ20A
- moved D3 30.8 mm to (144.3, 81.7), turned to 90 degrees
- moved C14 0.75 mm to (148.6, 84.5)
- moved C15 0.75 mm to (148.6, 81.5)
- moved D1 0.75 mm to (117.1, 80.7)
Connections:
- net Net-(D10-K) renamed /RPI_VBUS_K
- D1 pad 1: /POE_VP -> /POE_VP_F
- D2 pad 1: /POE_VP -> /POE_VP_F
- D4 pad 1: Net-(D4-K) -> /IC1_EED0_LED2
- D4 pad 2: /IC1_EED0_LED2 -> /J1_LED_OR_A
- R13 pad 2: GND -> /U2_PG
- R21 pad 2: GND -> +3V3
- R22 pad 2: GND -> +3V3
- R3 pad 1: Net-(D4-K) -> /J1_LED_OR_A
- R3 pad 2: GND -> +3V3
Routing:
- net /POE_VP_F: track 0.00 -> 46.2 mm, vias 0 -> 2
- net /POE_VP: track 41.2 -> 10.6 mm
- net Net-(D4-K): track 29.2 -> 0.00 mm, vias 2 -> 0
- net /J1_LED_OR_A: track 0.00 -> 25.4 mm, vias 0 -> 2
- net /U2_PG: track 4.15 -> 20.0 mm
- net +3V3: track 81.4 -> 87.6 mm, vias 12 -> 14
- net /POE_VP_A: track 0.00 -> 3.64 mm
- net GND: track 153.9 -> 150.4 mm, vias 96 -> 97
- net /IC1_EED0_LED2: track 67.9 -> 69.4 mm
- net /J6_DB_C: track 21.0 -> 20.3 mm
- net /J6_DA_C: track 14.4 -> 13.9 mm
Other:
- board text added: "POE VP"
- board text added: "Passive PoE 4-18Vdc > 20Vdc will cause permanent damage!"
- board text added: "^ (Check F2)"
