File: pizero-papoe/pizero-papoe.kicad_sch (KiCad schematic)
At the start: 67 parts, among them J1 RJ45-LED, P2 dnp-REF-182665-01, Q2 DMMT3906_Dual_PNP, Q3 Q_PMOS_GSD, T1 H2019FNL, U1 ENC28J60-I/ML, U2 TPS63070RNMR, U3 nostuff-AT24CS32-SSHM, U4 AP7365_SOT-23-5, Y1 25Mhz

Commit message: sch updates for RTL8153B and RJE7318800240
Parts:
- removed C11: 10uf, Capacitor_SMD:C_1206_3216Metric, symbol pizero-papoe-rescue:C
- removed C18, C21: 0.1uf, Capacitor_SMD:C_0603_1608Metric, symbol pizero-papoe-rescue:C
- removed C19, C20: 1uF, Capacitor_SMD:C_0603_1608Metric, symbol pizero-papoe-rescue:C_Small
- removed D7: LED Green, LED_SMD:LED_0603_1608Metric, symbol pizero-papoe-rescue:Led_Small
- removed H1, H2, H3, H4: hole-metalized-no4, pizero-poe-special:hole-m3, symbol pizero-papoe-rescue:hole-metalized-no4
- removed J1: RJ45-LED, pizero-poe-special:rj45-tyco-2-406549-7, symbol pizero-papoe-rescue:RJ45-LED
- removed P2: dnp-REF-182665-01, pizero-poe-special:Pin_Header_Straight_TH-SMT-NoPaste_2x20, symbol pizero-papoe-rescue:CONN_02X20
- removed R18: nostuff-1k, Resistor_SMD:R_0603_1608Metric, symbol pizero-papoe-rescue:R_Small
- removed R20, R23: nostuff-3.9k, Resistor_SMD:R_0603_1608Metric, symbol pizero-papoe-rescue:R_Small
- removed R24: 220, Resistor_SMD:R_0603_1608Metric, symbol pizero-papoe-rescue:R_Small
- removed R3: 1k, Resistor_SMD:R_0603_1608Metric, symbol pizero-papoe-rescue:R
- removed R8: 2.32k, Resistor_SMD:R_0603_1608Metric, symbol pizero-papoe-rescue:R
- removed U1: ENC28J60-I/ML, Package_DFN_QFN:QFN-28-1EP_6x6mm_P0.65mm_EP4.25x4.25mm, symbol pizero-papoe-rescue:ENC28J60-I/ML
- removed U3: nostuff-AT24CS32-SSHM, Package_SO:TSSOP-8_4.4x3mm_P0.65mm, symbol pizero-papoe-rescue:AT24CS32-SSHM
- removed U4: AP7365_SOT-23-5, Package_TO_SOT_SMD:SOT-23-5, symbol pizero-papoe-rescue:AP7365_SOT-23-5
- removed W1, W2: TEST_1P, TestPoint:TestPoint_Pad_D1.0mm, symbol pizero-papoe-rescue:TEST_1P
- added A1: Raspberry Pi Zero/W/2W, Raspberry_Pi_Zero_v.1.3_Hat:RPi_Zero_ZeroW_Zero2W_Hat_NoPads_NoHeader, symbol PiZeroHat:RPi_Zero_ZeroW_Zero2W_Hat_NoPads_NoHeader
- added C18, C21: 1nF, symbol pizero-papoe-rescue:C_Small
- added C19, C20, C32: 4.7uF, Capacitor_SMD:C_0603_1608Metric, symbol pizero-papoe-rescue:C
- added C25, C26, C27, C28, C29, C30, C31, C33, C35, C36, C41, C42: 0.1uf, Capacitor_SMD:C_0603_1608Metric, symbol pizero-papoe-rescue:C
- added C34: 1uF, Capacitor_SMD:C_0603_1608Metric, symbol pizero-papoe-rescue:C
- added C37, C38, C39, C40: 0.1uF 0201, symbol pizero-papoe-rescue:C_Small
- added IC1: RTL8153B-VB-CG, pizero-poe-special:RTL8153B-VB-CG_QFN40P500X500X90-41N-D, symbol pizero-papoe-special:RTL8153B-VB-CG
- added J2, J3, J4, J5: PogoPin_01x01, pizero-poe-special:PogoPin_CPG-04-TH-TR, symbol pizero-papoe-special:PogoPin_01x01
- added J6: RJ45_LED_AK_Shielded, symbol pizero-papoe-special:RJ45_LED_AK_Shielded
- added L3: 2.2uH, Inductor_SMD:L_Sunlord_SWPA4030S, symbol Device:L
- added P1: USB_C_Plug_USB3.0_9P, pizero-poe-special:USB_C_Plug_G-Switch_GT-USB-8016A_9P_TopMnt_Horizontal, symbol pizero-papoe-special:USB_C_Plug_USB3.0_9P
- added R10, R6, R7, R9: 75, Resistor_SMD:R_0603_1608Metric, symbol pizero-papoe-rescue:R
- added R11, R12: 22, Resistor_SMD:R_0603_1608Metric, symbol pizero-papoe-rescue:R
- added R18, R20: 22-dnp, Resistor_SMD:R_0603_1608Metric, symbol pizero-papoe-rescue:R
- added R23: 10k, Resistor_SMD:R_0603_1608Metric, symbol Device:R_Small
- added TR1: 30F-51NL, Transformer_SMD:Transformer_Ethernet_YDS_30F-51NL_SO-24_7.1x15.1mm, symbol Transformer:30F-51NL
- C17: value nostuff-0.1u -> 1nF; footprint Capacitor_SMD:C_0603_1608Metric -> (none); Type nostuff -> (none)
Connections:
- net +3V3: now also C25.1, C26.1, C27.1, C28.1, C29.1, C30.1, IC1.11 (AVDD33_1), IC1.20 (AVDD33_2), IC1.23 (DVDD33_1), IC1.33 (DVDD33_2), IC1.39 (AVDD33_3), IC1.40 (AVDD33_4), R23.1; no longer C10.1, C17.1, C7.1, C8.1, C9.1, R21.2, R22.2
- net GND: now also R21.2, R22.2, C18.2, C19.2, C20.2, C21.2, C25.2, C26.2, C27.2, C28.2, C29.2, C30.2, C31.2, C32.2, C33.2, C34.2, C35.2, C36.2, C41.2, C42.2, IC1.29 (GND), IC1.41 (EP), J5.1 (Pin_1); no longer C17.2
- net RPI_VBUS: now also C32.1, C33.1, IC1.21 (VDD5), J2.1 (Pin_1)
- net LEDA_A renamed J1_LED_GN_A
- net J1_LED_GN_A: now also J6.9
- net LEDB_A renamed J1_LED_YL_A
- net J1_LED_YL_A: now also J6.11
- net PHY_OSC1 renamed IC1_CKXTAL1
- net IC1_CKXTAL1: now also IC1.35 (CKXTAL1)
- net PHY_OSC2 renamed IC1_CKXTAL2
- net IC1_CKXTAL2: now also IC1.36 (CKXTAL2)
- net TPIN_T+: no longer names the net of T1.11 (RX+)
- net TPIN_T-: no longer names the net of T1.9 (RX-)
- net TPOUT_T+: no longer names the net of T1.16 (TX+)
- net TPOUT_T-: no longer names the net of T1.14 (TX-)
- new net: C19.1, C7.1, IC1.26 (VDDREG33), IC1.27 (VDDREG5)
- new net: IC1.28 (REGOUT), L3.2
- new net: P1.A1 (GND), P1.A12 (GND), P1.B1 (GND), P1.B12 (GND)
- new net: P1.A4 (VBUS), P1.A9 (VBUS), P1.B4 (VBUS), P1.B9 (VBUS)
- new net +1V0: C10.1, C20.1, C31.1, C36.1, C41.1, C42.1, C8.1, C9.1, IC1.14 (U3VDD10), IC1.19 (U2VDD10), IC1.3 (AVDD10_1), IC1.34 (DVDD10), IC1.37 (AVDD10_3), IC1.8 (AVDD10_2), L3.1
- new net DA_C: R6.1, TR1.15 (CT)
- new net DB_C: R7.1, TR1.18 (CT)
- new net DC_C: R9.1, TR1.21 (CT)
- new net DD_C: R10.1, TR1.24 (CT)
- new net IC1_DVDD10_UPS: C34.1, C35.1, IC1.22 (DVDD10_UPS)
- new net IC1_EECS: IC1.31 (EECS)
- new net IC1_EED0: IC1.24 (EEDO/LED2/SPISDO/LANW/AKEB/GPIO)
- new net IC1_EEDI_ENSWREG: IC1.25 (EEDI/SPISDI/ENSWREG), R23.2
- new net IC1_LED0_SPICSB: IC1.32 (LED0/SPICSB), J6.10
- new net IC1_LED1_SPISCK: IC1.30 (EESK/LED1/SPISCK), J6.12
- new net IC1_MDIN0: IC1.2 (MDIN0), TR1.11 (TD4+)
- new net IC1_MDIN1: IC1.5 (MDIN1), TR1.8 (TD3+)
- new net IC1_MDIN2: IC1.7 (MDIN2), TR1.5 (TD2+)
- new net IC1_MDIN3: IC1.10 (MDIN3), TR1.2 (TD1+)
- new net IC1_MDIP0: IC1.1 (MDIP0), TR1.12 (TD4-)
- new net IC1_MDIP1: IC1.4 (MDIP1), TR1.9 (TD3-)
- new net IC1_MDIP2: IC1.6 (MDIP2), TR1.6 (TD2-)
- new net IC1_MDIP3: IC1.9 (MDIP3), TR1.3 (TD1-)
- new net IC1_U2DM: IC1.17 (U2DM), R11.2, R18.2
- new net IC1_U2DP: IC1.18 (U2DP), R12.2, R20.2
- new net IC1_U3SSRX_C_N: C38.2, P1.B10 (RX1-)
- new net IC1_U3SSRX_C_P: C37.2, P1.B11 (RX1+)
- new net IC1_U3SSRX_N: C38.1, IC1.15 (U3SSRXN)
- new net IC1_U3SSRX_P: C37.1, IC1.16 (U3SSRXP)
- new net IC1_U3SSTX_C_N: C40.2, P1.A3 (TX1-)
- new net IC1_U3SSTX_C_P: C39.2, P1.A2 (TX1+)
- new net IC1_U3SSTX_N: C40.1, IC1.12 (U3SSTXN)
- new net IC1_U3SSTX_P: C39.1, IC1.13 (U3SSTXP)
- new net J1_1_DA_P: J6.1, TR1.13 (MX4-)
- new net J1_2_DA_N: J6.2, TR1.14 (MX4+)
- new net J1_3_DB_P: J6.3, TR1.16 (MX3-)
- new net J1_4_DC_P: J6.4, TR1.19 (MX2-)
- new net J1_5_DC_N: J6.5, TR1.20 (MX2+)
- new net J1_6_DB_N: J6.6, TR1.17 (MX3+)
- new net J1_7_DD_P: J6.7, TR1.22 (MX1-)
- new net J1_8_DD_N: J6.8, TR1.23 (MX1+)
- new net J1_CT_C: C17.2, R10.2, R6.2, R7.2, R9.2
- new net J1_SH_C: C17.1, C18.1, C21.1, J6.SH
- new net J4_U2DM: J3.1 (Pin_1), R11.1
- new net J5_U2DP: J4.1 (Pin_1), R12.1
- new net P1_U2DM: P1.A7 (D-), R18.1
- new net P1_U2DP: P1.A6 (D+), R20.1
- new net TR1_CT_1: TR1.10 (CT)
- new net TR1_CT_2: TR1.7 (CT)
- new net TR1_CT_3: TR1.4 (CT)
- new net TR1_CT_4: TR1.1 (CT)
- no-connect marks 6 -> 0
Other:
- note added: "Depop and R11 and R12 to use USB 2 on P1"
- note added: "ENSWREG: Power-on Latch: 3.3V = SW Reg En"
- note added: "In LAN disabled state, LED pin output voltage is 0v."
- note added: "LED Code 4: LED 2 (Left, 9-10): Green LED 1 (Right, 11-12): Yellow"
- note added: "RJE7318800240 RJ Connector is 11.75 mm tall to fit under SD Card"
- note added: "TODO: config EEPROM 93LC46 / MX25L1606E"
- note removed: "16-bit addressed I2C EEPROM, 32Kb+ Stores RPi HAT configuration."
- note removed: "Ethernet PHY"
- note removed: "Extra Linear Reg. for 3.3V Power ethernet phy whether we have PoE or not. Phy requires more power than allowed from RPi 3.3V."
- note removed: "Raspberry Pi Header"
- note removed: "TH Female Bottom or SMT Female Top Header SMT: Toby Electronics REF-182665-01/REF-182665-03 TH: Digikey 1528-1385-ND Pin #s Match RPi."
- moved on the sheet: C10, C2, C3, C7, C8, C9, L2, R14, R16, R17, R21, R22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

Commit message: complete RTL8153B sch
Parts:
- removed L2: BEAD, Resistor_SMD:R_0603_1608Metric, symbol pizero-papoe-rescue:INDUCTOR
- removed R10, R6, R7, R9: 75, Resistor_SMD:R_0603_1608Metric, symbol pizero-papoe-rescue:R
- removed R14, R16, R17, R26: 49.9, Resistor_SMD:R_0603_1608Metric, symbol pizero-papoe-rescue:R
- removed T1: H2019FNL, pizero-poe-special:Transformer_Pulse_H2019FNL, symbol pizero-papoe-rescue:H2019FNL
- added C11, C43, C44, C45, C46: 0.1uF, Capacitor_SMD:C_0201_0603Metric, symbol pizero-papoe-rescue:C_Small
- added D4: LED Orange, LED_SMD:LED_0603_1608Metric, symbol pizero-papoe-rescue:Led_Small
- added J1: PogoPin_01x01, pizero-poe-special:PogoPin_CPG-01-TH-TR, symbol pizero-papoe-special:PogoPin_01x01
- added R3: 1k, Resistor_SMD:R_0603_1608Metric, symbol pizero-papoe-rescue:R
- added U1: 93LC46B, Package_SO:SOIC-8_3.9x4.9mm_P1.27mm, symbol Memory_EEPROM:93LCxxA
- added U3: MX25L3233FM1, Package_SO:SOP-8_5.28x5.23mm_P1.27mm, symbol Memory_Flash:MX25L3233FM1
- C17: value 1nF -> 0.1uF; footprint (none) -> Capacitor_SMD:C_0201_0603Metric
- C18, C21: footprint (none) -> Capacitor_SMD:C_0603_1608Metric
- C2: value 16pf -> 30pf; LCSC (none) -> C501847; Mfg (none) -> FH; Mfg PN (none) -> 0603CG300F500NT
- C3: value 16pf -> 30pf
- C37, C38, C39, C40: footprint (none) -> Capacitor_SMD:C_0201_0603Metric
- D6: Digikey Part No 160-1183-1-ND -> (none); LCSC (none) -> C125093
- F1: footprint (none) -> pizero-poe-special:Fuse_2016_5041Metric
- IC1: footprint pizero-poe-special:RTL8153B-VB-CG_QFN40P500X500X90-41N-D -> Package_DFN_QFN:QFN-40-1EP_5x5mm_P0.4mm_EP3.6x3.6mm_ThermalVias
- J2, J3, J4, J5: footprint pizero-poe-special:PogoPin_CPG-04-TH-TR -> pizero-poe-special:PogoPin_CPG-01-TH-TR; Mfg PN CPG-04-TH-TR -> CPG-01-TH-TR
- J6: footprint (none) -> pizero-poe-special:RJ45_Amphenol_RJE7318800xxx0x
- R21, R22: value 549 -> 1k
- Y1: CL (none) -> 20pF
Connections:
- net DA_C is gone; now on net J6_DA_C: TR1.15 (CT)
- net DB_C is gone; now on net J6_DB_C: TR1.18 (CT)
- net SPARE_PAIR_1 is gone; now on net J6_DD_C: D2.3 (~{2})
- net SPARE_PAIR_2 is gone; now on net J6_DC_C: D2.2 (~{1})
- net TR1_CT_1 is gone; now on net TR1_CT: TR1.10 (CT)
- net TR1_CT_2 is gone; now on net TR1_CT: TR1.7 (CT)
- net TR1_CT_3 is gone; now on net TR1_CT: TR1.4 (CT)
- net TR1_CT_4 is gone; now on net TR1_CT: TR1.1 (CT)
- net +3V3: now also U1.8 (VCC), U3.3 (~{WP}/SIO2), U3.7 (~{HOLD}/SIO3), U3.8 (VCC)
- net GND: now also C17.1, C11.1, J1.1 (Pin_1), R3.2, U1.5 (GND), U3.4 (GND)
- net IC1_EECS: now also U1.1 (CS)
- net IC1_EEDI_ENSWREG: now also U1.3 (DI), U3.5 (SI/SIO0)
- net IC1_LED0_SPICSB: now also U3.1 (~{CS})
- net IC1_LED1_SPISCK: now also U1.2 (SCLK), U3.6 (SCLK)
- net J1_SH_C: now also C43.2, C44.2, C45.2, C46.2; no longer C17.1
- net RPI_VBUS: now also C19.1, C7.1, IC1.26 (VDDREG33), IC1.27 (VDDREG5)
- net IC1_REGOUT: now reaches IC1.28 (REGOUT), L3.2
- net DATA_PAIR_1 renamed J6_DA_C
- net J6_DA_C: now also C43.1
- net DATA_PAIR_2 renamed J6_DB_C
- net J6_DB_C: now also C44.1
- net DC_C renamed J6_DC_C
- net J6_DC_C: now also C45.1
- net DD_C renamed J6_DD_C
- net J6_DD_C: now also C46.1
- net IC1_EED0 renamed IC1_EED0_LED2
- net IC1_EED0_LED2: now also D4.2 (A), U1.4 (DO), U3.2 (SO/SIO1)
- net J1_1_DA_P renamed J6_1_DA_P
- net J1_2_DA_N renamed J6_2_DA_N
- net J1_3_DB_P renamed J6_3_DB_P
- net J1_4_DC_P renamed J6_4_DC_P
- net J1_5_DC_N renamed J6_5_DC_N
- net J1_6_DB_N renamed J6_6_DB_N
- net J1_7_DD_P renamed J6_7_DD_P
- net J1_8_DD_N renamed J6_8_DD_N
- net J1_CT_C renamed TR1_CT
- net TR1_CT: now also C11.2
- new net: D4.1 (K), R3.1
Other:
- note added: "30pf = 2*(CL-Cstray) using 5pf for Cstray"
- note added: "93LC46 DS: ORG can only be floated for clock speeds of 1 MHz or less for the x16 memory organization. ORG=0 is x8 organizataion ORG=1 is x16 organization - 93LC46B is always x16"
- note added: "93LC46 EEPROM used in https://github.com/OLIMEX/USB-GIGABIT/blob/master/ HARDWARE/USB-GIGABIT-Rev.C/USB-GIGABIT_Rev_C.pdf"
- note added: "IEEE PoE may send a detection voltage of 2.7-10.1 V looking for a 25kohm load at this end."
- note added: "Ideal Diode for RPi 5V Source Q1: Low Rds PFET like DMP3099L. 3A, 99mΩ @ 4.5V Vgs. Q2: Matched PNP pair. Current mirror comparator pulls Q3 gate low (on) when USB_VBUS_RVP > USB_VBUS."
- note added: "SPI Flash MX25L1606E used on https://www.96boards.org/documentation/consumer/ dragonboard/db4/hardware-docs/files/db4-sch.pdf"
- note removed: "Ideal Diode for RPi 5V Source Q1: Low Rds PFET like DMP3099L. 3A, 99mΩ @ 4.5V Vgs. Q2: Matched PNP pair. Current mirror comparator pulls Q1 gate low (on) when USB_VBUS_RVP > USB_VBUS."
- note removed: "Open drain LEDs set default to full-duplex on reset."
- note removed: "RJ45 & Transformer"
- note removed: "TODO: config EEPROM 93LC46 / MX25L1606E"
- moved on the sheet: J3, J4, R11, R12

Commit message: pcb routing for RTL8153B and RJE7318800240
Parts:
- removed C1, C22: 0.1uf 100V, Capacitor_SMD:C_0603_1608Metric, symbol pizero-papoe-rescue:C
- added D6, D7, D8, D9: TPD1E01B04-dnp, Diode_SMD:D_0402_1005Metric, symbol Device:D_TVS_Small_Filled
- added R6: 5.1k, Resistor_SMD:R_0603_1608Metric, symbol Device:R_Small
- added R7: 10k, Resistor_SMD:R_0603_1608Metric, symbol Device:R_Small
- added U4: WE-TVS-82400102-dnp, Package_TO_SOT_SMD:SOT-23-6, symbol Power_Protection:WE-TVS-82400102
- C11, C17, C43, C44, C45, C46: footprint Capacitor_SMD:C_0201_0603Metric -> Capacitor_SMD:C_0603_1608Metric
- L3: footprint Inductor_SMD:L_Sunlord_SWPA4030S -> Inductor_SMD:L_1008_2520Metric; JLCPCB Part # LCSC -> (none); LCSC (none) -> C2986800; Mfg Coilcraft -> DDY; Mfg 2 Sunlord -> APV; Mfg 2 Part No SWPA4030S1R5NT -> ANR252010T2R2M; Mfg Part No XFL4020-152ME -> SFE252010S-2R2M-HF
- P1, R18, R20: now not fitted
- renumbered D6 to D5
Connections:
- net +3V3: now also R7.2
- net +5V: now also P1.A4 (VBUS), P1.A9 (VBUS), P1.B4 (VBUS), P1.B9 (VBUS), U4.5
- net GND: now also P1.A1 (GND), P1.A12 (GND), P1.B1 (GND), P1.B12 (GND), P1.S1 (SHIELD), D6.2 (A2), D7.2 (A2), D8.2 (A2), D9.2 (A2), R6.2, U4.2
- net P1_U2DP: now also U4.3, U4.4
- net IC1_RST: now reaches IC1.38 (RSET)
- net IC1_RST: now also R7.1
- net P1_CC: now reaches P1.A5 (CC)
- net P1_CC: now also R6.1
- net IC1_MDIN0 renamed IC1_MDI0_N
- net IC1_MDIN1 renamed IC1_MDI1_N
- net IC1_MDIN2 renamed IC1_MDI2_N
- net IC1_MDIN3 renamed IC1_MDI3_N
- net IC1_MDIP0 renamed IC1_MDI0_P
- net IC1_MDIP1 renamed IC1_MDI1_P
- net IC1_MDIP2 renamed IC1_MDI2_P
- net IC1_MDIP3 renamed IC1_MDI3_P
- net IC1_U2DM renamed IC1_U2DN
- net IC1_U3SSRX_C_N renamed P1_U3SSRX_N
- net P1_U3SSRX_N: now also D9.1 (A1)
- net IC1_U3SSRX_C_P renamed P1_U3SSRX_P
- net P1_U3SSRX_P: now also D8.1 (A1)
- net IC1_U3SSTX_C_N renamed P1_U3SSTX_N
- net P1_U3SSTX_N: now also D7.1 (A1)
- net IC1_U3SSTX_C_P renamed P1_U3SSTX_P
- net P1_U3SSTX_P: now also D6.1 (A1)
- net J4_U2DM renamed A1_U2DN
- net J5_U2DP renamed A1_U2DP
- net J6_1_DA_P renamed J6_DA_P
- net J6_2_DA_N renamed J6_DA_N
- net J6_3_DB_P renamed J6_DB_P
- net J6_4_DC_P renamed J6_DC_P
- net J6_5_DC_N renamed J6_DC_N
- net J6_6_DB_N renamed J6_DB_N
- net J6_7_DD_P renamed J6_DD_P
- net J6_8_DD_N renamed J6_DD_N
- net P1_U2DM renamed P1_U2DN
- net P1_U2DN: now also U4.1, U4.6
- no-connect marks 0 -> 1
Other:
- note added: "DA: 1&2"
- note added: "DB: 3&6"
- note added: "DC: 4&5"
- note added: "DD: 7&8"
- note added: "RTL8153B DS Max Power ~400mW or ~80mA @ 5V Request 500mA @ 5V"
- moved on the sheet: A1, J1, J2, J3, J4, J5, R11, R12, U1

Commit message: pizero-papoe sch pcb fixes and cleanup
Parts:
- removed C19: 4.7uF, Capacitor_SMD:C_0603_1608Metric, symbol pizero-papoe-rescue:C
- added C1: 0.1uf, Capacitor_SMD:C_0603_1608Metric, symbol pizero-papoe-rescue:C
- added C19, C22: 1uF, Capacitor_SMD:C_0603_1608Metric, symbol pizero-papoe-rescue:C_Small
- added D10: LED Green, LED_SMD:LED_0603_1608Metric, symbol pizero-papoe-rescue:Led_Small
- added R8: 1k, Resistor_SMD:R_0603_1608Metric, symbol pizero-papoe-rescue:R_Small
- added TP1: VBUS, TestPoint:TestPoint_Pad_D1.5mm, symbol Connector:TestPoint
- added TP2: GND, TestPoint:TestPoint_Pad_D1.5mm, symbol Connector:TestPoint
- added TP3: 3V3, TestPoint:TestPoint_Pad_D1.5mm, symbol Connector:TestPoint
- C18, C21: value 1nF -> 1uF
- C29: value 0.1uf -> 4.7uF
Connections:
- net +3V3: now also IC1.26 (VDDREG33), C1.1, TP3.1
- net GND: now also C1.2, C19.2, C22.2, R8.2, TP2.1; no longer P1.S1 (SHIELD)
- net RPI_VBUS: now also D10.2 (A), TP1.1; no longer IC1.26 (VDDREG33)
- new net: D10.1 (K), R8.1
- new net P1_SH: C19.1, C22.1, P1.SH1 (SHIELD)
Other:
- note added: "Backup 3V3 for RTL8153B Pads for Sparkfun BabyBuck AP63203 or similar."
- note added: "RTL8153B Power Tree: In: VDDREG5 (Pin 27) - accepts 3.3V or 5V? In: VDDREG33 (Pin 26) - accepts 3.3V? Out: AVDD33 (Pin 20) - feeds AVDD33 and DVDD33 pins Out: REGOUT @ 1V (Pin 28) - feeds AVDD10 and DVDD10 pins Out: DVDD10_UPS (Pin 22) - decoupling only"
- company: OpenFet -> (none)
- title: Raspberry Pi - Power Over Ethernet & PHY -> PiZero Passive PoE & USB Ethernet

Commit message: pizero-papoe pcb sch bom tweaks for r1
Parts:
- added D11: LED Green, LED_SMD:LED_0603_1608Metric, symbol pizero-papoe-rescue:Led_Small
- added F2: JFC1206-1250FS, Fuse:Fuse_1206_3216Metric, symbol Device:Polyfuse
- added R9: 10k, Resistor_SMD:R_0603_1608Metric, symbol Device:R_Small
- A1: LCSC (none) -> --
- C1, C10, C25, C26, C27, C28, C30, C31, C33, C35, C36, C41, C42, C7, C8, C9: value 0.1uf -> 0.1uF; LCSC (none) -> C6119867
- C11, C17, C43, C44, C45, C46: LCSC (none) -> C6119867
- C13: LCSC (none) -> C882505
- C14, C15, C16, C6: LCSC (none) -> C6119965
- C18, C19, C21, C22, C34: LCSC (none) -> C5673
- C2: value 30pf -> 30pF
- C20, C29, C32: LCSC (none) -> C6119855
- C23, C24: value nostuff-330-1200uF -> 330-1200uF-dnp; now not fitted
- C3: value 30pf -> 30pF; LCSC (none) -> C501847
- C37, C38, C39, C40: LCSC (none) -> C6119757
- C4: LCSC C108079 -> C6119867
- C5: LCSC C2178233 -> C6119965
- D2: LCSC (none) -> C2488
- D3: value SMAJ58A -> SMAJ20A; LCSC C148209 -> C115250
- D7, D8, D9: LCSC (none) -> C779389
- IC1: LCSC (none) -> C2802072; Manufacturer_Name Realtek -> (none); Manufacturer_Part_Number RTL8153B-VB-CG -> (none); Mfg (none) -> Realtek; Mfg PN (none) -> RTL8153B-VB-CG
- J1, J2, J3, J4, J5: LCSC (none) -> --; Mfg PN CPG-01-TH-TR -> CPG-01-TH-B
- J6: LCSC (none) -> --; Mfg (none) -> Amphenol; Mfg PN (none) -> RJE7318800240
- L1: JLCPCB Part # LCSC -> (none); LCSC (none) -> C5127390; Mfg 2 Sunlord -> LanTu Micro; Mfg 2 Part No SWPA4030S1R5NT -> SNR4030-1R5MT
- R1: LCSC (none) -> C23198
- R11, R12: LCSC (none) -> C1203
- R13, R21, R22, R3, R8: LCSC (none) -> C21190
- R15, R2, R23, R5, R7: LCSC (none) -> C15401
- R19, R4: LCSC (none) -> C25600
- R6: LCSC (none) -> C26000
- TP1, TP2, TP3: now not fitted
- TR1: LCSC (none) -> C123168
- Y1: LCSC (none) -> C251592; LSCS C251592 -> (none); Mouser Part No. 774-445I23D25M00000 -> (none)
Connections:
- net +3V3: now also R21.2, R22.2, R3.2
- net GND: now also D11.1 (K); no longer R13.2, R21.2, R22.2, R3.2
- net IC1_EED0_LED2: now also D4.1 (K); no longer D4.2 (A)
- net POE_VP: now also F2.2; no longer D1.1 (V+), D2.1 (V+)
- net U2_PG: now also R13.2
- net RPI_VBUS_K: now reaches D10.1 (K), R8.1
- net J1_LED_OR_A: now reaches R3.1
- net J1_LED_OR_A: now also D4.2 (A); no longer D4.1 (K)
- new net POE_VP_A: D11.2 (A), R9.2
- new net POE_VP_F: D1.1 (V+), D2.1 (V+), F2.1, R9.1
Other:
- note added: "IEEE PoE may send a detection voltage of 2.7-10.1 V looking for a 25kohm load at this end. Protect against higher than 20V input reaching the TPS63070."
- note added: "Passive PoE (4.5-18V) -> 2A Buck-Boost (4-16V) -> 5V"
- note removed: "IEEE PoE may send a detection voltage of 2.7-10.1 V looking for a 25kohm load at this end."
- note removed: "Passive PoE (4-16V) -> 2A Buck-Boost -> 5V"
- moved on the sheet: D4, D5, R13, R8

Commit message: add pizero-papoe bom info and step export
Parts:
- U4: LCSC (none) -> C2827654; Mfg (none) -> WE; Mfg 2 (none) -> Tech Public; Mfg 2 PN (none) -> USBLC6-2SC6; Mfg PN (none) -> WE-TVS-82400102
Changed lines of the file:
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@@
+			)
+		)
+		(property "Mfg" "WE"
+			(at 83.82 130.81 0)
+			(effects
+				(font
+					(size 1.27 1.27)
+				)
+				(hide yes)
+			)
+		)
+		(property "Mfg PN" "WE-TVS-82400102"
+			(at 83.82 130.81 0)
+			(effects
+				(font
+					(size 1.27 1.27)
+				)
+				(hide yes)
+			)
+		)
+		(property "Mfg 2" "Tech Public"
+			(at 83.82 130.81 0)
+			(effects
+				(font
+					(size 1.27 1.27)
+				)
+				(hide yes)
+			)
+		)
+		(property "Mfg 2 PN" "USBLC6-2SC6"
+			(at 83.82 130.81 0)
+			(effects
+				(font
+					(size 1.27 1.27)
+				)
+				(hide yes)
+			)
+		)
+		(property "LCSC" "C2827654"
+			(at 83.82 130.81 0)
+			(effects
+				(font
+					(size 1.27 1.27)
+				)
+				(hide yes)
 			)
 		)
